File: strum2/strum2.brd (EAGLE design)
At the start: 164.8 x 99.1 mm, 97 parts, among them IC2 REG1117, IC3 74HC595D, IC4 74HC595D, SW1 12MMTACT_SMT, SW10 12MMTACT_SMT, SW11 12MMTACT_SMT, SW12 12MMTACT_SMT, SW13 12MMTACT_SMT, SW14 12MMTACT_SMT, SW15 12MMTACT_SMT, SW16 12MMTACT_SMT, SW17 12MMTACT_SMT, SW18 12MMTACT_SMT, SW19 12MMTACT_SMT, SW2 12MMTACT_SMT, SW20 12MMTACT_SMT, SW21 12MMTACT_SMT, SW22 12MMTACT_SMT, SW23 12MMTACT_SMT, SW24 12MMTACT_SMT, SW25 12MMTACT_SMT, SW26 12MMTACT_SMT, SW27 12MMTACT_SMT, SW28 12MMTACT_SMT, SW29 12MMTACT_SMT, SW3 12MMTACT_SMT, SW30 12MMTACT_SMT, SW31 12MMTACT_SMT, SW32 12MMTACT_SMT, SW33 12MMTACT_SMT, SW34 12MMTACT_SMT, SW35 12MMTACT_SMT, SW36 12MMTACT_SMT, SW4 12MMTACT_SMT, SW5 12MMTACT_SMT, SW6 12MMTACT_SMT, SW7 12MMTACT_SMT, SW8 12MMTACT_SMT, SW9 12MMTACT_SMT, U1 MCU-PIC16F1825-I/ST(TSSOP14)

Commit message: dasasddads
Parts:
- moved STYLUS1 76.6 mm to (151.4, 96.5)
- moved MIDI 20.7 mm to (74.9, 94.0)
- moved PWR 20.6 mm to (74.9, 97.2)
- moved STYLUS 11.6 mm to (86.4, 96.5)
- moved R3 9.53 mm to (69.8, 97.2)
- moved R8 7.78 mm to (69.8, 94.9)
- moved R4 7.73 mm to (69.8, 92.7)
- moved C2 3.31 mm to (59.1, 55.9), turned to 90 degrees
- moved C4 3.19 mm to (59.1, 76.2), turned to 90 degrees
- moved S37 2.47 mm to (62.2, 93.9), turned to 270 degrees
- moved IC4 1.27 mm to (62.2, 83.8)
Connections:
- removed net N$52: MIDI.C, R4.2
- removed net N$54: PWR.C, R8.1
- new net N$1: PWR.A, R8.2
- new net N$12: MIDI.A, R4.1
- net GND: now also MIDI.C, PWR.C; no longer R4.1, R8.2
- net RA2: now also IC4.11, IC4.12
- net RC2: now also R4.2; no longer MIDI.A
- net VCC: now also R8.1; no longer PWR.A
Routing:
- net RC1: track 28.3 -> 112.4 mm
- net N$34: track 0.00 -> 77.7 mm
- net N$27: track 0.00 -> 69.8 mm
- net VCC: track 70.2 -> 127.2 mm
- net RA2: track 4.33 -> 43.8 mm, vias 0 -> 3
- net N$28: track 0.00 -> 33.0 mm
- net N$38: track 0.00 -> 30.8 mm
- net RC0: track 8.56 -> 33.7 mm, vias 0 -> 2
- net RC5: track 0.00 -> 23.3 mm, vias 0 -> 1
- net N$22: track 0.00 -> 20.3 mm
- net CARRY: track 0.00 -> 17.6 mm, vias 0 -> 2
- net N$37: track 0.00 -> 17.5 mm
- net N$5: track 0.00 -> 16.0 mm
- net N$14: track 0.00 -> 15.8 mm
- net N$26: track 0.00 -> 14.3 mm
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- added copper zone on layer 1, net GND
Other:
- outline, holes or cut-outs redrawn

Commit message: asads
Parts:
- added STYLUS2, STYLUS3: M01PTH, SparkFun:1X01
- moved R1 5.08 mm to (15.2, 82.5), turned to 270 degrees
- moved STYLUS1 1.27 mm to (152.7, 96.5)
- moved MIDI_OUT 1.27 mm to (13.0, 91.4)
- moved R2 1.27 mm to (11.4, 82.5), turned to 270 degrees
- moved STYLUS 1.27 mm to (85.1, 96.5)
Connections:
- net RC1: now also STYLUS2.1, STYLUS3.1
Routing:
- net RA5: track 372.0 -> 384.5 mm
- net N$22: track 20.3 -> 11.7 mm
- net RA4: track 405.3 -> 399.3 mm
- net VCC: track 127.2 -> 132.2 mm
- net RC4: track 24.6 -> 29.2 mm
- net LINE5: track 165.5 -> 161.9 mm
- net RC1: track 112.4 -> 113.7 mm
- net N$48: track 3.23 -> 4.43 mm
- net LINE1: track 150.6 -> 151.5 mm
- net LINE4: track 162.3 -> 162.8 mm, vias 4 -> 2
- added copper zone on layer 16, net GND
Other:
- board size 164.8 x 99.1 mm -> 167.6 x 99.1 mm

Commit message: asddsa
Parts:
- renumbered S37 to MODE
Routing:
- net RA5: track 384.5 -> 382.6 mm
Other:
- board text added: "7"
- board text added: "A"
- board text added: "B"
- board text added: "C"
- board text added: "D"
- board text added: "D2 -D17"
- board text added: "E"
- board text added: "F"
- board text added: "G"
- board text added: "M"
- board text added: "m"
- board text removed: "+9V"
- board text removed: "GND"

Commit message: sdfsdf
Parts:
- removed U1: MCU-PIC16F1825-I/ST(TSSOP14), MCU-PIC16F1825-I_ST_TSSOP14_:TSSOP14-0.65-5X4.4MM
- added IC1: REG1117, burr-brown:SOT223
- C1, C2: device rcl:C0805 -> rcl:E2-5
- C5, C6: device rcl:E2-5 -> rcl:C0805
- IC2: value REG1117 -> MCU-PIC16F1825-I/ST(TSSOP14); device burr-brown:SOT223 -> MCU-PIC16F1825-I_ST_TSSOP14_:TSSOP14-0.65-5X4.4MM
- R5: value 10k -> 1k
- R8: value 1k -> 10k
- moved R5 71.4 mm to (69.8, 92.7), turned to 180 degrees
- moved R8 55.7 mm to (39.4, 48.3)
- moved C2 44.3 mm to (25.0, 84.2), turned to 180 degrees
- moved C7 36.3 mm to (59.1, 55.9), turned to 90 degrees
- moved C6 35.0 mm to (59.1, 76.2), turned to 90 degrees
- moved C4 25.4 mm to (34.4, 82.5), turned to 180 degrees
- moved C1 20.6 mm to (25.1, 89.9)
- moved C5 20.6 mm to (45.7, 91.3)
- moved IC3 20.3 mm to (62.2, 83.8)
- moved IC4 20.3 mm to (62.2, 63.5)
- moved R6 12.7 mm to (14.0, 48.3)
- moved R7 12.7 mm to (26.7, 48.3)
- moved IC2 11.4 mm to (45.7, 87.0)
- moved R1 3.81 mm to (11.4, 82.5)
- moved R2 3.81 mm to (15.2, 82.5)
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Connections:
- net CARRY: now also IC3.14, IC4.9; no longer IC3.9, IC4.14
- net GND: now also C1.-, C2.-, C5.1, C6.1, IC1.1, IC2.14, R8.1; no longer C1.1, C2.1, C5.-, C6.-, IC2.1, R5.1, U1.14
- net N$1: now also R4.2; no longer R8.2
- net N$10: now also IC4.5; no longer IC3.5
- net N$11: now also IC4.6; no longer IC3.6
- net N$12: now also R5.1; no longer R4.1
- net N$13: now also IC4.7; no longer IC3.7
- net N$14: now also IC3.15; no longer IC4.15
- net N$15: now also IC3.1; no longer IC4.1
- net N$16: now also IC3.2; no longer IC4.2
- net N$17: now also IC3.3; no longer IC4.3
- net N$18: now also IC3.4; no longer IC4.4
- net N$19: now also IC3.5; no longer IC4.5
- net N$20: now also IC3.6; no longer IC4.6
- net N$21: now also IC3.7; no longer IC4.7
- net N$44: now also R2.1; no longer R1.1
- net N$48: now also R1.2; no longer R2.2
- net N$5: now also IC4.15; no longer IC3.15
- net N$59: now also C2.+, C4.2, IC1.3; no longer C6.+, C7.2, IC2.3
- net N$6: now also IC4.1; no longer IC3.1
- net N$7: now also IC4.2; no longer IC3.2
- net N$8: now also IC4.3; no longer IC3.3
- net N$9: now also IC4.4; no longer IC3.4
- net RA0: now also IC2.13; no longer U1.13
- net RA1: now also IC2.12; no longer U1.12
- net RA2: now also IC2.11; no longer U1.11
- net RA3: now also IC2.4; no longer U1.4
- net RA4: now also IC2.3, R7.2; no longer R6.2, U1.3
- net RA5: now also IC2.2, R6.2; no longer R5.2, U1.2
- net RC0: now also IC2.10, IC4.14; no longer IC3.14, U1.10
- net RC1: now also IC2.9; no longer U1.9
- net RC2: now also IC2.8, R5.2; no longer R4.2, U1.8
- net RC3: now also IC2.7, R8.2; no longer R7.2, U1.7
- net RC4: now also IC2.6, R2.2; no longer R1.2, U1.6
- net RC5: now also IC2.5; no longer U1.5
- net VCC: now also C1.+, C5.2, C6.2, C7.2, IC1.2, IC2.1, R1.1, R4.1; no longer C1.2, C2.2, C4.2, C5.+, IC2.2, R2.1, R8.1, U1.1
Routing:
- net N$34: track 77.7 -> 82.8 mm
- net LINE13: track 134.1 -> 135.9 mm
- net LINE12: track 191.8 -> 193.3 mm
- net LINE11: track 162.5 -> 163.9 mm
- net LINE10: track 167.4 -> 168.5 mm
