File: strum2/strum2.sch (EAGLE design)
At the start: 97 parts, among them IC2 REG1117, IC3 74HC595D, IC4 74HC595D, SW1 12MMTACT_SMT, SW10 12MMTACT_SMT, SW11 12MMTACT_SMT, SW12 12MMTACT_SMT, SW13 12MMTACT_SMT, SW14 12MMTACT_SMT, SW15 12MMTACT_SMT, SW16 12MMTACT_SMT, SW17 12MMTACT_SMT, SW18 12MMTACT_SMT, SW19 12MMTACT_SMT, SW2 12MMTACT_SMT, SW20 12MMTACT_SMT, SW21 12MMTACT_SMT, SW22 12MMTACT_SMT, SW23 12MMTACT_SMT, SW24 12MMTACT_SMT, SW25 12MMTACT_SMT, SW26 12MMTACT_SMT, SW27 12MMTACT_SMT, SW28 12MMTACT_SMT, SW29 12MMTACT_SMT, SW3 12MMTACT_SMT, SW30 12MMTACT_SMT, SW31 12MMTACT_SMT, SW32 12MMTACT_SMT, SW33 12MMTACT_SMT, SW34 12MMTACT_SMT, SW35 12MMTACT_SMT, SW36 12MMTACT_SMT, SW4 12MMTACT_SMT, SW5 12MMTACT_SMT, SW6 12MMTACT_SMT, SW7 12MMTACT_SMT, SW8 12MMTACT_SMT, SW9 12MMTACT_SMT, U1 MCU-PIC16F1825-I/ST(TSSOP14)

Commit message: dasasddads
Connections:
- removed net N$52: MIDI.C, R4.2
- removed net N$54: PWR.C, R8.1
- new net N$1: PWR.A, R8.2
- new net N$12: MIDI.A, R4.1
- net GND: now also MIDI.C, PWR.C; no longer R4.1, R8.2
- net RA2: now also IC4A.RCK, IC4A.SCK
- net RC2: now also R4.2; no longer MIDI.A
- net VCC: now also R8.1; no longer PWR.A
Other:
- moved on the sheet: MIDI, PWR, R4, R8
Changed lines of the file:
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@@
 <instance part="STYLUS" gate="G$1" x="408.94" y="375.92" rot="R180"/>
 <instance part="R3" gate="G$1" x="314.96" y="358.14" rot="R90"/>
-<instance part="R4" gate="G$1" x="342.9" y="358.14" rot="R90"/>
-<instance part="MIDI" gate="G$1" x="322.58" y="386.08" rot="R90"/>
+<instance part="R4" gate="G$1" x="325.12" y="386.08" rot="R180"/>
+<instance part="MIDI" gate="G$1" x="335.28" y="386.08" rot="R90"/>
 <instance part="R5" gate="G$1" x="185.42" y="363.22" rot="R180"/>
 <instance part="R6" gate="G$1" x="185.42" y="358.14" rot="R180"/>
 <instance part="R7" gate="G$1" x="185.42" y="353.06" rot="R180"/>
 <instance part="D1" gate="G$1" x="147.32" y="406.4"/>
-<instance part="R8" gate="G$1" x="243.84" y="363.22" rot="R270"/>
-<instance part="PWR" gate="G$1" x="243.84" y="386.08"/>
+<instance part="R8" gate="G$1" x="243.84" y="386.08" rot="R270"/>
+<instance part="PWR" gate="G$1" x="243.84" y="363.22"/>
 <instance part="ONOFF" gate="1" x="165.1" y="408.94" rot="R180"/>
 <instance part="S37" gate="S" x="297.18" y="419.1"/>
@@
 <pinref part="IC3" gate="A" pin="QH*"/>
 <junction x="261.62" y="314.96"/>
+<junction x="381" y="337.82"/>
 </segment>
 </net>
 <net name="VCC" class="0">
 <segment>
-<wire x1="243.84" y1="393.7" x2="243.84" y2="388.62" width="0.1524" layer="91"/>
 <wire x1="254" y1="393.7" x2="243.84" y2="393.7" width="0.1524" layer="91"/>
 <wire x1="254" y1="391.16" x2="254" y2="393.7" width="0.1524" layer="91"/>
@@
 <wire x1="215.9" y1="403.86" x2="215.9" y2="408.94" width="0.1524" layer="91"/>
 <wire x1="223.52" y1="403.86" x2="223.52" y2="408.94" width="0.1524" layer="91"/>
-<junction x="243.84" y="388.62"/>
 <junction x="254" y="393.7"/>
 <junction x="271.78" y="393.7"/>
@@
 <junction x="274.32" y="309.88"/>
 <junction x="223.52" y="408.94"/>
-<pinref part="PWR" gate="G$1" pin="A"/>
 <pinref part="C3" gate="G$1" pin="1"/>
 <pinref part="ICSP" gate="G$1" pin="2"/>
@@
 <junction x="215.9" y="408.94"/>
 <label x="274.32" y="393.7" size="1.778" layer="95"/>
+<pinref part="R8" gate="G$1" pin="1"/>
+<wire x1="243.84" y1="393.7" x2="243.84" y2="391.16" width="0.1524" layer="91"/>
+<junction x="388.62" y="337.82"/>
 </segment>
 <segment>
@@
 <junction x="251.46" y="340.36"/>
 <label x="302.26" y="370.84" size="1.778" layer="95"/>
+<pinref part="IC4" gate="A" pin="SCK"/>
+<junction x="386.08" y="337.82"/>
+<pinref part="IC4" gate="A" pin="RCK"/>
+<junction x="393.7" y="337.82"/>
 </segment>
 <segment>
@@
 <wire x1="261.62" y1="342.9" x2="261.62" y2="353.06" width="0.1524" layer="91"/>
 <wire x1="261.62" y1="353.06" x2="314.96" y2="353.06" width="0.1524" layer="91"/>
-<wire x1="314.96" y1="353.06" x2="342.9" y2="353.06" width="0.1524" layer="91"/>
-<wire x1="342.9" y1="353.06" x2="353.06" y2="353.06" width="0.1524" layer="91"/>
 <wire x1="353.06" y1="353.06" x2="403.86" y2="353.06" width="0.1524" layer="91"/>
 <wire x1="403.86" y1="353.06" x2="411.48" y2="353.06" width="0.1524" layer="91"/>
@@
 <wire x1="198.12" y1="353.06" x2="198.12" y2="358.14" width="0.1524" layer="91"/>
 <wire x1="198.12" y1="391.16" x2="198.12" y2="363.22" width="0.1524" layer="91"/>
-<wire x1="243.84" y1="358.14" x2="243.84" y2="353.06" width="0.1524" layer="91"/>
 <wire x1="261.62" y1="363.22" x2="261.62" y2="416.56" width="0.1524" layer="91"/>
 <wire x1="261.62" y1="416.56" x2="261.62" y2="419.1" width="0.1524" layer="91"/>
@@
 <junction x="353.06" y="353.06"/>
 <junction x="314.96" y="353.06"/>
-<junction x="342.9" y="353.06"/>
 <junction x="198.12" y="358.14"/>
 <junction x="198.12" y="363.22"/>
-<junction x="243.84" y="353.06"/>
 <junction x="198.12" y="391.16"/>
 <junction x="198.12" y="353.06"/>
 <junction x="358.14" y="396.24"/>
-<junction x="243.84" y="358.14"/>
 <junction x="261.62" y="416.56"/>
 <junction x="261.62" y="363.22"/>
@@
 <pinref part="ICSP" gate="G$1" pin="3"/>
 <pinref part="R3" gate="G$1" pin="1"/>
-<pinref part="R4" gate="G$1" pin="1"/>
 <pinref part="R5" gate="G$1" pin="1"/>
 <pinref part="R6" gate="G$1" pin="1"/>
 <pinref part="R7" gate="G$1" pin="1"/>
-<pinref part="R8" gate="G$1" pin="2"/>
 <pinref part="S37" gate="S" pin="1"/>
 <pinref part="S37" gate="S" pin="2"/>
@@
 <wire x1="198.12" y1="396.24" x2="198.12" y2="391.16" width="0.1524" layer="91"/>
 <label x="274.32" y="363.22" size="1.778" layer="95"/>
+<pinref part="PWR" gate="G$1" pin="C"/>
+<wire x1="243.84" y1="358.14" x2="243.84" y2="353.06" width="0.1524" layer="91"/>
+<junction x="243.84" y="353.06"/>
+<wire x1="314.96" y1="353.06" x2="342.9" y2="353.06" width="0.1524" layer="91"/>
+<pinref part="MIDI" gate="G$1" pin="C"/>
+<wire x1="342.9" y1="353.06" x2="353.06" y2="353.06" width="0.1524" layer="91"/>
+<wire x1="340.36" y1="386.08" x2="342.9" y2="386.08" width="0.1524" layer="91"/>
+<wire x1="342.9" y1="386.08" x2="342.9" y2="353.06" width="0.1524" layer="91"/>
+<junction x="342.9" y="353.06"/>
+<junction x="403.86" y="337.82"/>
 </segment>
 <segment>
@@
 <segment>
 <wire x1="307.34" y1="386.08" x2="320.04" y2="386.08" width="0.1524" layer="91"/>
-<junction x="320.04" y="386.08"/>
-<pinref part="MIDI" gate="G$1" pin="A"/>
 <label x="302.26" y="386.08" size="1.778" layer="95"/>
+<pinref part="R4" gate="G$1" pin="2"/>
 </segment>
 <segment>
@@
 <wire x1="302.26" y1="436.88" x2="309.88" y2="436.88" width="0.1524" layer="91"/>
 <label x="309.88" y="436.88" size="1.778" layer="95"/>
-</segment>
-</net>
-<net name="N$52" class="0">
-<segment>
-<wire x1="327.66" y1="386.08" x2="342.9" y2="386.08" width="0.1524" layer="91"/>
-<wire x1="342.9" y1="386.08" x2="342.9" y2="363.22" width="0.1524" layer="91"/>
-<junction x="342.9" y="363.22"/>
-<junction x="327.66" y="386.08"/>
-<pinref part="MIDI" gate="G$1" pin="C"/>
-<pinref part="R4" gate="G$1" pin="2"/>
-</segment>
-</net>
-<net name="N$54" class="0">
-<segment>
-<wire x1="243.84" y1="381" x2="243.84" y2="368.3" width="0.1524" layer="91"/>
-<junction x="243.84" y="381"/>
-<junction x="243.84" y="368.3"/>
-<pinref part="PWR" gate="G$1" pin="C"/>
-<pinref part="R8" gate="G$1" pin="1"/>
 </segment>
 </net>
@@
 </segment>
 </net>
+<net name="N$1" class="0">
+<segment>
+<pinref part="R8" gate="G$1" pin="2"/>
+<pinref part="PWR" gate="G$1" pin="A"/>
+<wire x1="243.84" y1="381" x2="243.84" y2="365.76" width="0.1524" layer="91"/>
+</segment>
+</net>
+<net name="N$12" class="0">
+<segment>
+<pinref part="R4" gate="G$1" pin="1"/>
+<pinref part="MIDI" gate="G$1" pin="A"/>
+<wire x1="330.2" y1="386.08" x2="332.74" y2="386.08" width="0.1524" layer="91"/>
+</segment>
+</net>

Commit message: asads
Parts:
- added STYLUS2, STYLUS3: M01PTH, SparkFun:M01PTH
Connections:
- net RC1: now also STYLUS2.1, STYLUS3.1
Changed lines of the file:
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@@
 <part name="SW35" library="jason_eagle6" deviceset="12MMTACT_SMT" device=""/>
 <part name="SW36" library="jason_eagle6" deviceset="12MMTACT_SMT" device=""/>
+<part name="STYLUS2" library="SparkFun" deviceset="M01" device="PTH"/>
+<part name="STYLUS3" library="SparkFun" deviceset="M01" device="PTH"/>
 </parts>
 <sheets>
@@
 <instance part="SW35" gate="G$1" x="406.4" y="147.32"/>
 <instance part="SW36" gate="G$1" x="429.26" y="147.32"/>
+<instance part="STYLUS2" gate="G$1" x="408.94" y="381" rot="R180"/>
+<instance part="STYLUS3" gate="G$1" x="408.94" y="386.08" rot="R180"/>
 </instances>
 <busses>
@@
 <pinref part="STYLUS1" gate="G$1" pin="1"/>
 <wire x1="391.16" y1="370.84" x2="401.32" y2="370.84" width="0.1524" layer="91"/>
-</segment>
-<segment>
+<pinref part="STYLUS3" gate="G$1" pin="1"/>
+<wire x1="401.32" y1="386.08" x2="391.16" y2="386.08" width="0.1524" layer="91"/>
+<wire x1="391.16" y1="386.08" x2="391.16" y2="381" width="0.1524" layer="91"/>
+<pinref part="STYLUS2" gate="G$1" pin="1"/>
+<wire x1="391.16" y1="381" x2="391.16" y2="375.92" width="0.1524" layer="91"/>
+<wire x1="401.32" y1="381" x2="391.16" y2="381" width="0.1524" layer="91"/>
+<junction x="391.16" y="381"/>
+</segment>
+<segment>

Commit message: asddsa
Parts:
- renumbered S37 to MODE
Changed lines of the file:
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@@
 <part name="PWR" library="led" deviceset="LED" device="CHIPLED_0805"/>
 <part name="ONOFF" library="SparkFun" deviceset="SWITCH-SPST" device="PTH"/>
-<part name="S37" library="SparkFun" deviceset="TAC_SWITCH" device="PTH"/>
+<part name="MODE" library="SparkFun" deviceset="TAC_SWITCH" device="PTH"/>
 <part name="STYLUS1" library="SparkFun" deviceset="M01" device="PTH"/>
 <part name="C1" library="rcl" deviceset="C-EU" device="C0805"/>
@@
 <instance part="PWR" gate="G$1" x="243.84" y="363.22"/>
 <instance part="ONOFF" gate="1" x="165.1" y="408.94" rot="R180"/>
-<instance part="S37" gate="S" x="297.18" y="419.1"/>
+<instance part="MODE" gate="S" x="297.18" y="419.1"/>
 <instance part="STYLUS1" gate="G$1" x="408.94" y="370.84" rot="R180"/>
 <instance part="C1" gate="G$1" x="274.32" y="327.66"/>
@@
 <pinref part="R6" gate="G$1" pin="1"/>
 <pinref part="R7" gate="G$1" pin="1"/>
-<pinref part="S37" gate="S" pin="1"/>
-<pinref part="S37" gate="S" pin="2"/>
+<pinref part="MODE" gate="S" pin="1"/>
+<pinref part="MODE" gate="S" pin="2"/>
 <pinref part="C1" gate="G$1" pin="1"/>
 <pinref part="C2" gate="G$1" pin="1"/>
@@
 <junction x="302.26" y="419.1"/>
 <junction x="302.26" y="416.56"/>
-<pinref part="S37" gate="S" pin="3"/>
-<pinref part="S37" gate="S" pin="4"/>
+<pinref part="MODE" gate="S" pin="3"/>
+<pinref part="MODE" gate="S" pin="4"/>
 <label x="302.26" y="393.7" size="1.778" layer="95"/>
 </segment>

Commit message: sdfsdf
Parts:
- removed U1: MCU-PIC16F1825-I/ST(TSSOP14), MCU-PIC16F1825-I_ST_TSSOP14_:MCU-PIC16F1825-I/ST(TSSOP14)
- added IC1: REG1117, burr-brown:REG1117
- C1, C2: device rcl:C-EUC0805 -> rcl:CPOL-EUE2-5
- C5, C6: device rcl:CPOL-EUE2-5 -> rcl:C-EUC0805
- IC2: value REG1117 -> MCU-PIC16F1825-I/ST(TSSOP14); device burr-brown:REG1117 -> MCU-PIC16F1825-I_ST_TSSOP14_:MCU-PIC16F1825-I/ST(TSSOP14)
- R5: value 10k -> 1k
- R8: value 1k -> 10k
Connections:
- net CARRY: now also IC3A.SER, IC4A.QH*; no longer IC3A.QH*, IC4A.SER
- net GND: now also C1.-, C2.-, C5.1, C6.1, IC1.GND, IC2.VSS, R8.1; no longer C1.1, C2.1, C5.-, C6.-, IC2.GND, R5.1, U1.VSS
- net N$1: now also R4.2; no longer R8.2
- net N$10: now also IC4A.QF; no longer IC3A.QF
- net N$11: now also IC4A.QG; no longer IC3A.QG
- net N$12: now also R5.1; no longer R4.1
- net N$13: now also IC4A.QH; no longer IC3A.QH
- net N$14: now also IC3A.QA; no longer IC4A.QA
- net N$15: now also IC3A.QB; no longer IC4A.QB
- net N$16: now also IC3A.QC; no longer IC4A.QC
- net N$17: now also IC3A.QD; no longer IC4A.QD
- net N$18: now also IC3A.QE; no longer IC4A.QE
- net N$19: now also IC3A.QF; no longer IC4A.QF
- net N$20: now also IC3A.QG; no longer IC4A.QG
- net N$21: now also IC3A.QH; no longer IC4A.QH
- net N$44: now also R2.1; no longer R1.1
- net N$48: now also R1.2; no longer R2.2
- net N$5: now also IC4A.QA; no longer IC3A.QA
- net N$59: now also C2.+, C4.2, IC1.VIN; no longer C6.+, C7.2, IC2.VIN
- net N$6: now also IC4A.QB; no longer IC3A.QB
- net N$7: now also IC4A.QC; no longer IC3A.QC
- net N$8: now also IC4A.QD; no longer IC3A.QD
- net N$9: now also IC4A.QE; no longer IC3A.QE
- net RA0: now also IC2.RA0; no longer U1.RA0
- net RA1: now also IC2.RA1; no longer U1.RA1
- net RA2: now also IC2.RA2; no longer U1.RA2
- net RA3: now also IC2.RA3; no longer U1.RA3
- net RA4: now also IC2.RA4, R7.2; no longer R6.2, U1.RA4
- net RA5: now also IC2.RA5, R6.2; no longer R5.2, U1.RA5
- net RC0: now also IC2.RC0, IC4A.SER; no longer IC3A.SER, U1.RC0
- net RC1: now also IC2.RC1; no longer U1.RC1
- net RC2: now also IC2.RC2, R5.2; no longer R4.2, U1.RC2
- net RC3: now also IC2.RC3, R8.2; no longer R7.2, U1.RC3
- net RC4: now also IC2.RC4, R2.2; no longer R1.2, U1.RC4
- net RC5: now also IC2.RC5; no longer U1.RC5
- net VCC: now also C1.+, C5.2, C6.2, C7.2, IC1.VOUT, IC2.VDD, R1.1, R4.1; no longer C1.2, C2.2, C4.2, C5.+, IC2.VOUT, R2.1, R8.1, U1.VDD
Other:
- moved on the sheet: C4, C7, IC3, IC3P, IC4, IC4P, R1, R2, R4, R5, R6, R7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

Commit message: asasas
Parts:
- removed IC2: MCU-PIC16F1825-I/ST(TSSOP14), MCU-PIC16F1825-I_ST_TSSOP14_:MCU-PIC16F1825-I/ST(TSSOP14)
- added D18, D19: TS4148, jason_eagle6:TS4148
- added IC5: PIC16F1825SO14, jasons_stuff:PIC16F1825SO14
Connections:
- new net N$24: D18.A, STYLUS2.1, STYLUS3.1
- new net N$25: D19.A, STYLUS.1, STYLUS1.1
- net GND: now also IC5.VSS; no longer IC2.VSS
- net RA0: now also IC5.RA0/ICSPDAT; no longer IC2.RA0
- net RA1: now also IC5.RA1/ICPCLK; no longer IC2.RA1
- net RA2: now also IC5.RA2/INT; no longer IC2.RA2
- net RA3: now also IC5.RA3/MCLR#/VPP; no longer IC2.RA3
- net RA4: now also IC5.RA4/SDO; no longer IC2.RA4
- net RA5: now also IC5.RA5; no longer IC2.RA5
- net RC0: now also IC5.RCO/SCL/SCK; no longer IC2.RC0
- net RC1: now also D18.C, D19.C, IC5.RC1/SDA/SDI; no longer IC2.RC1, STYLUS.1, STYLUS1.1, STYLUS2.1, STYLUS3.1
- net RC2: now also IC5.RC2; no longer IC2.RC2
- net RC3: now also IC5.RC3/SS#; no longer IC2.RC3
- net RC4: now also IC5.RC4/TX; no longer IC2.RC4
- net RC5: now also IC5.RC5/RX; no longer IC2.RC5
- net VCC: now also IC5.VDD; no longer IC2.VDD

Commit message: REV 1
Parts:
- renumbered IC5 to IC2
Connections:
- net LINE1: now also D4.C; no longer D2.C
- net LINE10: now also D13.C; no longer D11.C
- net LINE11: now also D14.C; no longer D12.C
- net LINE12: now also D15.C; no longer D13.C
- net LINE13: now also D16.C; no longer D14.C
- net LINE14: now also D17.C; no longer D15.C
- net LINE15: now also D18.C; no longer D16.C
- net LINE16: now also D19.C; no longer D17.C
- net LINE2: now also D5.C; no longer D3.C
- net LINE3: now also D6.C; no longer D4.C
- net LINE4: now also D7.C; no longer D5.C
- net LINE5: now also D8.C; no longer D6.C
- net LINE6: now also D9.C; no longer D7.C
- net LINE7: now also D10.C; no longer D8.C
- net LINE8: now also D11.C; no longer D9.C
- net LINE9: now also D12.C; no longer D10.C
- net N$10: now also D9.A; no longer D7.A
- net N$11: now also D10.A; no longer D8.A
- net N$13: now also D11.A; no longer D9.A
- net N$14: now also D12.A; no longer D10.A
- net N$15: now also D13.A; no longer D11.A
- net N$16: now also D14.A; no longer D12.A
- net N$17: now also D15.A; no longer D13.A
- net N$18: now also D16.A; no longer D14.A
- net N$19: now also D17.A; no longer D15.A
- net N$20: now also D18.A; no longer D16.A
- net N$21: now also D19.A; no longer D17.A
- net N$24: now also D2.A; no longer D18.A
- net N$25: now also D3.A; no longer D19.A
- net N$5: now also D4.A; no longer D2.A
- net N$6: now also D5.A; no longer D3.A
- net N$7: now also D6.A; no longer D4.A
- net N$8: now also D7.A; no longer D5.A
- net N$9: now also D8.A; no longer D6.A
- net RC1: now also D2.C, D3.C; no longer D18.C, D19.C
Other:
- note added: "(c) J HOTCHKISS"
- note added: "17 NOV 2022"
- note added: "CC-NC-BY-SA"
- note added: "LE GRAND STRUM V1"
- moved on the sheet: D10, D11, D12, D13, D14, D15, D16, D17, D18, D19, D2, D3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
