File: le_grand_strum/le_grand_strum.brd (EAGLE design)
At the start: 167.6 x 99.1 mm, 101 parts, among them IC1 REG1117, IC2 PIC16F1825SO14, IC3 74HC595D, IC4 74HC595D, SW1 12MMTACT_SMT, SW10 12MMTACT_SMT, SW11 12MMTACT_SMT, SW12 12MMTACT_SMT, SW13 12MMTACT_SMT, SW14 12MMTACT_SMT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

Commit message: FINAL V1
Other:
- board size 167.6 x 99.1 mm -> 186.9 x 99.1 mm
