File: le_grand_strum/le_grand_strum.brd (EAGLE design)
At the start: 186.9 x 104.1 mm, 101 parts, among them IC1 REG1117, IC2 PIC16F1825SO14, IC3 74HC595D, IC4 74HC595D

Commit message: VERSION 3
ground midi out pin 2
Connections:
- net GND: now also MIDI_OUT.2
Other:
- board text added: "LE GRAND STRUM REV3 hotchk155/2024"
- board text removed: "LE GRAND STRUM REV2 hotchk155/2023"
Changed lines of the file:
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@@
 <wire x1="167.592" y1="101.539" x2="167.592" y2="0.066" width="0.3048" layer="102"/>
 <circle x="43.053" y="98.044" radius="0.359209375" width="0.3048" layer="21"/>
-<text x="142.371" y="86.773" size="2.54" layer="22" font="vector" ratio="20" rot="SMR0">LE GRAND STRUM REV2
-hotchk155/2023</text>
+<text x="142.371" y="86.773" size="2.54" layer="22" font="vector" ratio="20" rot="SMR0">LE GRAND STRUM REV3
+hotchk155/2024</text>
 <wire x1="2.54" y1="48.5775" x2="15.24" y2="48.5775" width="0.4064" layer="21"/>
 <wire x1="15.24" y1="48.5775" x2="15.24" y2="32.385" width="0.4064" layer="21"/>
@@
 <via x="78.994" y="89.789" extent="1-16" drill="0.6"/>
 <contactref element="IC2" pad="14"/>
+<contactref element="MIDI_OUT" pad="2"/>
 </signal>
 <signal name="RC0">
