File: le_grand_strum_stencil/le_grand_strum_stencil.brd (EAGLE design)
At the start: 193 x 104.1 mm, 100 parts, among them IC1 REG1117, IC2 PIC16F1825SO14, IC3 74HC595D, IC4 74HC595D, SW1 12MMTACT_SMT, SW10 12MMTACT_SMT, SW11 12MMTACT_SMT, SW12 12MMTACT_SMT, SW13 12MMTACT_SMT, SW14 12MMTACT_SMT, SW15 12MMTACT_SMT, SW16 12MMTACT_SMT, SW17 12MMTACT_SMT, SW18 12MMTACT_SMT, SW19 12MMTACT_SMT, SW2 12MMTACT_SMT, SW20 12MMTACT_SMT, SW21 12MMTACT_SMT, SW22 12MMTACT_SMT, SW23 12MMTACT_SMT, SW24 12MMTACT_SMT, SW25 12MMTACT_SMT, SW26 12MMTACT_SMT, SW27 12MMTACT_SMT, SW28 12MMTACT_SMT, SW29 12MMTACT_SMT, SW3 12MMTACT_SMT, SW30 12MMTACT_SMT, SW31 12MMTACT_SMT, SW32 12MMTACT_SMT, SW33 12MMTACT_SMT, SW34 12MMTACT_SMT, SW35 12MMTACT_SMT, SW36 12MMTACT_SMT, SW4 12MMTACT_SMT, SW5 12MMTACT_SMT, SW6 12MMTACT_SMT, SW7 12MMTACT_SMT, SW8 12MMTACT_SMT, SW9 12MMTACT_SMT

Commit message: stencil
Parts:
- removed MIDI_OUT: DIN5PIN", jasons_stuff:TRUCONN90
- removed SW1, SW10, SW11, SW12, SW13, SW14, SW15, SW16, SW17, SW18, SW19, SW2, SW20, SW21, SW22, SW23, SW24, SW25, SW26, SW27, SW28, SW29, SW3, SW30, SW31, SW32, SW33, SW34, SW35, SW36, SW4, SW5, SW6, SW7, SW8, SW9: 12MMTACT_SMT, jason_eagle6:12MMTACT_SMT
- moved 14 3.59 mm to (148.3, 54.9)
- moved 16 3.59 mm to (158.5, 54.9)
- moved D11 3.59 mm to (72.4, 72.4)
- moved D12 3.59 mm to (72.4, 74.9)
- moved D14 3.59 mm to (72.4, 80.0)
- moved D16 3.59 mm to (72.4, 85.1)
- moved D18 3.59 mm to (72.4, 90.2)
- moved D9 3.59 mm to (72.4, 67.3)
- moved MODE 3.59 mm to (64.7, 96.5)
- moved STYLUS2 3.59 mm to (90.2, 99.1)
- moved C2 3.59 mm to (27.6, 86.7)
- moved R1 3.59 mm to (14.0, 85.1)
- moved R2 3.59 mm to (17.8, 85.1)
- moved 1 3.59 mm to (82.3, 54.9)
- moved 2 3.59 mm to (87.4, 54.9)
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Connections:
- net LINE1: no longer SW1.B1, SW1.B2, SW13.B1, SW13.B2, SW25.B1, SW25.B2
- net LINE10: no longer SW10.B1, SW10.B2, SW22.B1, SW22.B2, SW34.B1, SW34.B2
- net LINE11: no longer SW11.B1, SW11.B2, SW23.B1, SW23.B2, SW35.B1, SW35.B2
- net LINE12: no longer SW12.B1, SW12.B2, SW24.B1, SW24.B2, SW36.B1, SW36.B2
- net LINE2: no longer SW14.B1, SW14.B2, SW2.B1, SW2.B2, SW26.B1, SW26.B2
- net LINE3: no longer SW15.B1, SW15.B2, SW27.B1, SW27.B2, SW3.B1, SW3.B2
- net LINE4: no longer SW16.B1, SW16.B2, SW28.B1, SW28.B2, SW4.B1, SW4.B2
- net LINE5: no longer SW17.B1, SW17.B2, SW29.B1, SW29.B2, SW5.B1, SW5.B2
- net LINE6: no longer SW18.B1, SW18.B2, SW30.B1, SW30.B2, SW6.B1, SW6.B2
- net LINE7: no longer SW19.B1, SW19.B2, SW31.B1, SW31.B2, SW7.B1, SW7.B2
- net LINE8: no longer SW20.B1, SW20.B2, SW32.B1, SW32.B2, SW8.B1, SW8.B2
- net LINE9: no longer SW21.B1, SW21.B2, SW33.B1, SW33.B2, SW9.B1, SW9.B2
- net N$44: no longer MIDI_OUT.5
- net N$48: no longer MIDI_OUT.4
- net RA4: no longer SW13.A1, SW13.A2, SW14.A1, SW14.A2, SW15.A1, SW15.A2, SW16.A1, SW16.A2, SW17.A1, SW17.A2, SW18.A1, SW18.A2, SW19.A1, SW19.A2, SW20.A1, SW20.A2, SW21.A1, SW21.A2, SW22.A1, SW22.A2, SW23.A1, SW23.A2, SW24.A1, SW24.A2
- net RA5: no longer SW1.A1, SW1.A2, SW10.A1, SW10.A2, SW11.A1, SW11.A2, SW12.A1, SW12.A2, SW2.A1, SW2.A2, SW3.A1, SW3.A2, SW4.A1, SW4.A2, SW5.A1, SW5.A2, SW6.A1, SW6.A2, SW7.A1, SW7.A2, SW8.A1, SW8.A2, SW9.A1, SW9.A2
- net RC3: no longer SW25.A1, SW25.A2, SW26.A1, SW26.A2, SW27.A1, SW27.A2, SW28.A1, SW28.A2, SW29.A1, SW29.A2, SW30.A1, SW30.A2, SW31.A1, SW31.A2, SW32.A1, SW32.A2, SW33.A1, SW33.A2, SW34.A1, SW34.A2, SW35.A1, SW35.A2, SW36.A1, SW36.A2
Routing:
- net RA5: track 383.5 -> 403.5 mm, vias 12 -> 0
- net RC3: track 406.5 -> 416.1 mm, vias 13 -> 0
- net RA4: track 399.4 -> 408.2 mm, vias 13 -> 0
- net LINE7: track 154.3 -> 160.1 mm, vias 1 -> 2
- net N$28: track 33.0 -> 37.1 mm
- net LINE8: track 157.4 -> 161.0 mm
- net N$29: track 1.91 -> 0.00 mm
- net LINE12: track 193.3 -> 191.5 mm
- net LINE9: track 164.0 -> 165.8 mm
- net LINE6: track 160.8 -> 159.8 mm
- net N$33: track 3.18 -> 3.81 mm
- net LINE5: track 161.9 -> 162.5 mm
- net LINE1: track 151.5 -> 151.0 mm, vias 1 -> 0
- net LINE4: track 162.8 -> 163.3 mm
- net LINE3: track 162.7 -> 163.1 mm, vias 2 -> 1
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Other:
- board size 193 x 104.1 mm -> 197.5 x 113.3 mm
- board text added: "(c) 2023 sixty four pixels ltd"
- board text added: "LE GRAND STRUM REV2 hotchk155/2023"
- board text removed: "(c) 2022 sixty four pixels ltd"
- board text removed: "7"
- board text removed: "A"
- board text removed: "B"
- board text removed: "C"
- board text removed: "D"
- board text removed: "E"
- board text removed: "F"
- board text removed: "G"
- board text removed: "LE GRAND STRUM PCB REV1 hotchk155/2022"
- board text removed: "M"
- board text removed: "m"
- board text removed: "six4pix.com/strum"
